File: board_v2/BlackMagicProbe.kicad_sch (KiCad schematic)
At the start: 65 parts

Commit message: Clean up kicad5 files in board_v2
Parts:
- C1, C10, C11, C12, C13, C14, C15, C16, C17, C18, C5, C7, C8, C9: value (none) -> 100nF; footprint (none) -> Capacitor_SMD:C_0603_1608Metric_Pad1.05x0.95mm_HandSolder
- C2, C3: value (none) -> 18pF; footprint (none) -> Capacitor_SMD:C_0603_1608Metric_Pad1.05x0.95mm_HandSolder
- C4, C6: value (none) -> 4.7uF; footprint (none) -> Capacitor_SMD:C_0603_1608Metric_Pad1.05x0.95mm_HandSolder
- D1: renamed from D?; value (none) -> Green; footprint (none) -> LED_SMD:LED_0805_2012Metric
- D2, D3: renamed from D?; value (none) -> Yellow; footprint (none) -> LED_SMD:LED_0805_2012Metric
- D4: renamed from D?; value (none) -> Red; footprint (none) -> LED_SMD:LED_0805_2012Metric
- J1: value (none) -> DX07S016JA; footprint (none) -> sft:USB_C_JAE_DX07S0116JA1
- JP3, JP4, JP5, JP6, JP7, JP8, JP9: renamed from JP?; value (none) -> Jumper_NC_Small; footprint (none) -> sft:Jumper_2.54mm
- Q1, Q2: value (none) -> N-Channel; footprint (none) -> Package_TO_SOT_SMD:SOT-323_SC-70
- R1, R5, R7, R9: value (none) -> 10k; footprint (none) -> Resistor_SMD:R_0603_1608Metric_Pad1.05x0.95mm_HandSolder
- R10: renamed from R?; value (none) -> 15k; footprint (none) -> Resistor_SMD:R_0603_1608Metric_Pad1.05x0.95mm_HandSolder
- R11, R20, R21: renamed from R?; value (none) -> 1k5; footprint (none) -> Resistor_SMD:R_0603_1608Metric_Pad1.05x0.95mm_HandSolder
- R12, R13, R14, R15, R16, R17, R18, R19: value (none) -> 100; footprint (none) -> Resistor_SMD:R_0603_1608Metric_Pad1.05x0.95mm_HandSolder
- R2: value (none) -> 1k5; footprint (none) -> Resistor_SMD:R_0603_1608Metric_Pad1.05x0.95mm_HandSolder
- R3, R4: value (none) -> 22; footprint (none) -> Resistor_SMD:R_0603_1608Metric_Pad1.05x0.95mm_HandSolder
- R6, R70, R71, R8: value (none) -> 4k7; footprint (none) -> Resistor_SMD:R_0603_1608Metric_Pad1.05x0.95mm_HandSolder
- SW2: renamed from SW?; value (none) -> SW_Push; footprint (none) -> Button_Switch_THT:SW_PUSH_6mm_H4.3mm
- U1: value (none) -> STM32F103CBTx; footprint (none) -> Package_QFP:LQFP-48_7x7mm_P0.5mm
- U2, U3, U5, U6: value (none) -> SN74LVC2T45DCT; footprint (none) -> sft:TI-R-PDSO-G8
- U4: value (none) -> USBLC6-4SC6; footprint (none) -> Package_TO_SOT_SMD:SOT-23-6
- X1: value (none) -> SFT_DEBUG_CONNECTOR-SELF; footprint (none) -> Connector:Tag-Connect_TC2050-IDC-FP_2x05_P1.27mm_Vertical
- Y1: value (none) -> 8.000 MHz; footprint (none) -> Crystal:Crystal_HC49-4H_Vertical
- gave numbers to parts that had none: 1
