File: board_v2/OutputInterface.kicad_sch (KiCad schematic)
At the start: 149 parts

Commit message: Clean up kicad5 files in board_v2
Parts:
- C19, C20, C21, C22, C23, C24, C25: renamed from C?; value (none) -> 100nF; footprint (none) -> Capacitor_SMD:C_0603_1608Metric_Pad1.05x0.95mm_HandSolder
- D10, D11, D14, D22, D23, D24, D25, D9: renamed from D?; value (none) -> Yellow; footprint (none) -> LED_SMD:LED_0805_2012Metric
- D12, D13, D17, D19, D21, D5, D7: renamed from D?; value (none) -> Red; footprint (none) -> LED_SMD:LED_0805_2012Metric
- D15, D18, D20, D6, D8: renamed from D?; value (none) -> Green; footprint (none) -> LED_SMD:LED_0805_2012Metric
- D16, D26: renamed from D?; value (none) -> 4.7V; footprint (none) -> Diode_SMD:D_MiniMELF_Handsoldering
- D27, D29, D38: renamed from D?; value (none) -> 24V ESD; footprint (none) -> Resistor_SMD:R_0603_1608Metric_Pad1.05x0.95mm_HandSolder
- D30, D31, D32, D33, D34, D35, D36, D37: value (none) -> 1N4148WS; footprint (none) -> Diode_SMD:D_SOD-323
- FB1, FB2, FB3: value (none) -> 30Ω@100MHz; footprint (none) -> Resistor_SMD:R_0603_1608Metric_Pad1.05x0.95mm_HandSolder
- J10, J11, J12, J3, J4, J5, J6, J7, J8, J9: renamed from J?; value (none) -> Conn_01x04_Male; footprint (none) -> Connector_PinHeader_2.54mm:PinHeader_1x04_P2.54mm_Vertical
- J13, J14, J15, J16, J17: value (none) -> Conn_01x01_Female; footprint (none) -> sft:Connector_Banana_SKS_BIL20
- JP1, JP10, JP11, JP12, JP13, JP14, JP15, JP16, JP17, JP18, JP19: renamed from JP?; value (none) -> Jumper_NC_Small; footprint (none) -> sft:Jumper_2.54mm
- R22: renamed from R?; value (none) -> 50mOhm; footprint (none) -> Resistor_SMD:R_2010_5025Metric_Pad1.52x2.65mm_HandSolder
- R23, R36, R38, R43, R53, R55: renamed from R?; value (none) -> 33k; footprint (none) -> Resistor_SMD:R_0603_1608Metric_Pad1.05x0.95mm_HandSolder
- R24: renamed from R?; value (none) -> 30k; footprint (none) -> Resistor_SMD:R_0603_1608Metric_Pad1.05x0.95mm_HandSolder
- R25: renamed from R?; value (none) -> 27k; footprint (none) -> Resistor_SMD:R_0603_1608Metric_Pad1.05x0.95mm_HandSolder
- R26: renamed from R?; value (none) -> 18k; footprint (none) -> Resistor_SMD:R_0603_1608Metric_Pad1.05x0.95mm_HandSolder
- R27: renamed from R?; value (none) -> 75k; footprint (none) -> Resistor_SMD:R_0603_1608Metric_Pad1.05x0.95mm_HandSolder
- R28: renamed from R?; value (none) -> 12k; footprint (none) -> Resistor_SMD:R_0603_1608Metric_Pad1.05x0.95mm_HandSolder
- R29: renamed from R?; value (none) -> 1k8; footprint (none) -> Resistor_SMD:R_0603_1608Metric_Pad1.05x0.95mm_HandSolder
- R30: renamed from R?; value (none) -> 1k2; footprint (none) -> Resistor_SMD:R_0603_1608Metric_Pad1.05x0.95mm_HandSolder
- R31, R32, R33, R46, R47, R48, R49: renamed from R?; value (none) -> 100k; footprint (none) -> Resistor_SMD:R_0603_1608Metric_Pad1.05x0.95mm_HandSolder
- R34, R81: renamed from R?; value (none) -> 200; footprint (none) -> Resistor_SMD:R_0603_1608Metric_Pad1.05x0.95mm_HandSolder
- R35, R37, R39, R40, R41, R42, R44, R45, R52, R54, R56, R57, R58, R59, R60: renamed from R?; value (none) -> 3k3; footprint (none) -> Resistor_SMD:R_0603_1608Metric_Pad1.05x0.95mm_HandSolder
- R50, R51, R61, R62: renamed from R?; value (none) -> 10k; footprint (none) -> Resistor_SMD:R_0603_1608Metric_Pad1.05x0.95mm_HandSolder
- R63, R64, R65, R66, R67, R68, R69: renamed from R?; value (none) -> 1M; footprint (none) -> Resistor_SMD:R_0603_1608Metric_Pad1.05x0.95mm_HandSolder
- SW1: renamed from SW?; value (none) -> SW_Push; footprint (none) -> Button_Switch_THT:SW_PUSH_6mm_H4.3mm
- U10, U11, U12, U8, U9: renamed from U?; value (none) -> TS339; footprint (none) -> Package_SO:TSSOP-14_4.4x5mm_P0.65mm
- U13, U14: value (none) -> USBLC6-4SC6; footprint (none) -> Package_TO_SOT_SMD:SOT-23-6
- U7: renamed from U?; value (none) -> INA240A1; footprint (none) -> Package_SO:TSSOP-8_4.4x3mm_P0.65mm
- X2: renamed from X?; value (none) -> SFT debugport; footprint (none) -> Connector_IDC:IDC-Header_2x05_P2.54mm_Vertical
- X3: value (none) -> ARM debugport; footprint (none) -> Connector_IDC:IDC-Header_2x03_P2.54mm_Vertical
