File: board_v2/UserInterface.kicad_sch (KiCad schematic)
At the start: 6 parts

Commit message: Clean up kicad5 files in board_v2
Parts:
- JP20, JP21, JP22, JP23: value (none) -> SolderJumper_2_Bridged; footprint (none) -> Jumper:SolderJumper-2_P1.3mm_Bridged_RoundedPad1.0x1.5mm
- SW3: value (none) -> K1-1504SA-03; footprint (none) -> sft:K1-1504SA-03
- X4: renamed from X?; value (none) -> Blue; footprint (none) -> sft:OLED_128x64_096in
Changed lines of the file:
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@@
       (effects (font (size 1.524 1.524)))
     )
-    (property "Value" "" (id 1) (at 181.61 66.5226 0)
+    (property "Value" "K1-1504SA-03" (id 1) (at 181.61 66.5226 0)
       (effects (font (size 1.524 1.524)))
     )
-    (property "Footprint" "" (id 2) (at 182.88 81.28 0)
+    (property "Footprint" "sft:K1-1504SA-03" (id 2) (at 182.88 81.28 0)
       (effects (font (size 1.524 1.524)) hide)
     )
@@
   (symbol (lib_id "power:GND") (at 201.93 91.44 0) (unit 1)
     (in_bom yes) (on_board yes)
-    (property "Reference" "#PWR?" (id 0) (at 201.93 97.79 0)
+    (property "Reference" "#PWR0238" (id 0) (at 201.93 97.79 0)
       (effects (font (size 1.27 1.27)) hide)
     )
-    (property "Value" "" (id 1) (at 202.057 95.8342 0))
+    (property "Value" "GND" (id 1) (at 202.057 95.8342 0))
     (property "Footprint" "" (id 2) (at 201.93 91.44 0)
       (effects (font (size 1.27 1.27)) hide)
@@
     (in_bom yes) (on_board yes)
     (property "Reference" "JP20" (id 0) (at 71.12 73.533 0))
-    (property "Value" "" (id 1) (at 71.12 75.8444 0))
-    (property "Footprint" "" (id 2) (at 71.12 78.74 0)
+    (property "Value" "SolderJumper_2_Bridged" (id 1) (at 71.12 75.8444 0))
+    (property "Footprint" "Jumper:SolderJumper-2_P1.3mm_Bridged_RoundedPad1.0x1.5mm" (id 2) (at 71.12 78.74 0)
       (effects (font (size 1.27 1.27)) hide)
     )
@@
     (in_bom yes) (on_board yes)
     (property "Reference" "JP21" (id 0) (at 71.12 88.9 0))
-    (property "Value" "" (id 1) (at 71.12 86.36 0))
-    (property "Footprint" "" (id 2) (at 71.12 83.82 0)
+    (property "Value" "SolderJumper_2_Bridged" (id 1) (at 71.12 86.36 0))
+    (property "Footprint" "Jumper:SolderJumper-2_P1.3mm_Bridged_RoundedPad1.0x1.5mm" (id 2) (at 71.12 83.82 0)
       (effects (font (size 1.27 1.27)) hide)
     )
@@
     (in_bom yes) (on_board yes)
     (property "Reference" "JP23" (id 0) (at 88.9 93.98 0))
-    (property "Value" "" (id 1) (at 88.9 96.52 0))
-    (property "Footprint" "" (id 2) (at 88.9 99.06 0)
+    (property "Value" "SolderJumper_2_Bridged" (id 1) (at 88.9 96.52 0))
+    (property "Footprint" "Jumper:SolderJumper-2_P1.3mm_Bridged_RoundedPad1.0x1.5mm" (id 2) (at 88.9 99.06 0)
       (effects (font (size 1.27 1.27)) hide)
     )
@@
     (in_bom yes) (on_board yes)
     (property "Reference" "JP22" (id 0) (at 88.9 67.31 0))
-    (property "Value" "" (id 1) (at 88.9 64.77 0))
-    (property "Footprint" "" (id 2) (at 88.9 62.23 0)
+    (property "Value" "SolderJumper_2_Bridged" (id 1) (at 88.9 64.77 0))
+    (property "Footprint" "Jumper:SolderJumper-2_P1.3mm_Bridged_RoundedPad1.0x1.5mm" (id 2) (at 88.9 62.23 0)
       (effects (font (size 1.27 1.27)) hide)
     )
@@
   (symbol (lib_id "sft:OLED_I2C_128x64") (at 102.87 81.28 0) (unit 1)
     (in_bom yes) (on_board yes)
-    (property "Reference" "X?" (id 0) (at 118.8212 79.9338 0)
+    (property "Reference" "X4" (id 0) (at 118.8212 79.9338 0)
       (effects (font (size 1.524 1.524)) (justify left))
     )
-    (property "Value" "" (id 1) (at 118.8212 82.6262 0)
+    (property "Value" "Blue" (id 1) (at 118.8212 82.6262 0)
       (effects (font (size 1.524 1.524)) (justify left))
     )
-    (property "Footprint" "" (id 2) (at 102.87 81.28 0)
+    (property "Footprint" "sft:OLED_128x64_096in" (id 2) (at 102.87 81.28 0)
       (effects (font (size 1.524 1.524)) hide)
     )
@@
   (symbol (lib_id "power:GND") (at 82.55 101.6 0) (unit 1)
     (in_bom yes) (on_board yes)
-    (property "Reference" "#PWR?" (id 0) (at 82.55 107.95 0)
+    (property "Reference" "#PWR0236" (id 0) (at 82.55 107.95 0)
       (effects (font (size 1.27 1.27)) hide)
     )
-    (property "Value" "" (id 1) (at 82.677 105.9942 0))
+    (property "Value" "GND" (id 1) (at 82.677 105.9942 0))
     (property "Footprint" "" (id 2) (at 82.55 101.6 0)
       (effects (font (size 1.27 1.27)) hide)
@@
   (symbol (lib_id "power:+5V") (at 82.55 59.69 0) (unit 1)
     (in_bom yes) (on_board yes)
-    (property "Reference" "#PWR?" (id 0) (at 82.55 63.5 0)
+    (property "Reference" "#PWR0237" (id 0) (at 82.55 63.5 0)
       (effects (font (size 1.27 1.27)) hide)
     )
-    (property "Value" "" (id 1) (at 82.931 55.2958 0))
+    (property "Value" "+5V" (id 1) (at 82.931 55.2958 0))
     (property "Footprint" "" (id 2) (at 82.55 59.69 0)
       (effects (font (size 1.27 1.27)) hide)
