File: board_v2/board.kicad_sch (KiCad schematic)
At the start: 13 parts

Commit message: Clean up kicad5 files in board_v2
Parts:
- FID1, FID2, FID3, FID4, FID5, FID6, FID7, FID8: value (none) -> Fiducial; footprint (none) -> Fiducial:Fiducial_1mm_Mask2mm
- H1, H2, H3, H4: value (none) -> MountingHole_Pad; footprint (none) -> MountingHole:MountingHole_3.2mm_M3_Pad_Via
- LOGO1: value (none) -> Logo; footprint (none) -> sft:LOGO_CU_070
